File: 2057-ICE40HX4K-TQ144-breakout.sch (KiCad schematic (older format))
At the start: 73 parts, among them J1 Conn_02x30_Odd_Even, J2 Conn_02x30_Odd_Even, J3 RaspberryPI-B+header, J4 0548190519, J5 RaspberryPI-B+header, J6 Conn_02x08_Odd_Even, J7 Conn_02x01, J8 Micro_SD_Card_Det, U1 ICE40HX4K-TQ144, U2 AZ1117CH-3.3TRG1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

Commit message: Add Digikey info for ordering Diodes and LEDs
Parts:
- D1, D11, D12: Digi-Key_PN (none) -> 1N4448WSF-7DICT-ND; MPN (none) -> 1N4448WSF-7; Manufacturer (none) -> Diodes Incorporated
- D10, D2, D3, D4, D5, D6, D7, D8, D9: Description (none) -> Green LED; Digi-Key_PN (none) -> B1911PG--20D000514U1930; MPN (none) -> B1911PG--20D000514U1930; Manufacturer (none) -> Harvatek Corporation
Changed lines of the file:
@@
 F 2 "Diode_SMD:D_0603_1608Metric_Pad1.05x0.95mm_HandSolder" H 10250 1300 50  0001 C CNN
 F 3 "~" H 10250 1300 50  0001 C CNN
+F 4 "1N4448WSF-7DICT-ND" H 10250 1300 50  0001 C CNN "Digi-Key_PN"
+F 5 "1N4448WSF-7" H 10250 1300 50  0001 C CNN "MPN"
+F 6 "Diodes Incorporated" H 10250 1300 50  0001 C CNN "Manufacturer"
 	1    10250 1300
 	0    -1   -1   0
@@
 F 2 "LED_SMD:LED_0603_1608Metric_Pad1.05x0.95mm_HandSolder" H 14500 3500 50  0001 C CNN
 F 3 "~" H 14500 3500 50  0001 C CNN
+F 4 "Green LED" H 14500 3500 50  0001 C CNN "Description"
+F 5 "B1911PG--20D000514U1930" H 14500 3500 50  0001 C CNN "Digi-Key_PN"
+F 6 "B1911PG--20D000514U1930" H 14500 3500 50  0001 C CNN "MPN"
+F 7 "Harvatek Corporation" H 14500 3500 50  0001 C CNN "Manufacturer"
 	1    14500 3500
 	1    0    0    -1
@@
 F 2 "LED_SMD:LED_0603_1608Metric_Pad1.05x0.95mm_HandSolder" H 11400 4100 50  0001 C CNN
 F 3 "~" H 11400 4100 50  0001 C CNN
+F 4 "Green LED" H 11400 4100 50  0001 C CNN "Description"
+F 5 "B1911PG--20D000514U1930" H 11400 4100 50  0001 C CNN "Digi-Key_PN"
+F 6 "B1911PG--20D000514U1930" H 11400 4100 50  0001 C CNN "MPN"
+F 7 "Harvatek Corporation" H 11400 4100 50  0001 C CNN "Manufacturer"
 	1    11400 4100
 	1    0    0    -1
@@
 F 2 "LED_SMD:LED_0603_1608Metric_Pad1.05x0.95mm_HandSolder" H 11400 4350 50  0001 C CNN
 F 3 "~" H 11400 4350 50  0001 C CNN
+F 4 "Green LED" H 11400 4350 50  0001 C CNN "Description"
+F 5 "B1911PG--20D000514U1930" H 11400 4350 50  0001 C CNN "Digi-Key_PN"
+F 6 "B1911PG--20D000514U1930" H 11400 4350 50  0001 C CNN "MPN"
+F 7 "Harvatek Corporation" H 11400 4350 50  0001 C CNN "Manufacturer"
 	1    11400 4350
 	1    0    0    -1
@@
 F 2 "LED_SMD:LED_0603_1608Metric_Pad1.05x0.95mm_HandSolder" H 11400 4600 50  0001 C CNN
 F 3 "~" H 11400 4600 50  0001 C CNN
+F 4 "Green LED" H 11400 4600 50  0001 C CNN "Description"
+F 5 "B1911PG--20D000514U1930" H 11400 4600 50  0001 C CNN "Digi-Key_PN"
+F 6 "B1911PG--20D000514U1930" H 11400 4600 50  0001 C CNN "MPN"
+F 7 "Harvatek Corporation" H 11400 4600 50  0001 C CNN "Manufacturer"
 	1    11400 4600
 	1    0    0    -1
@@
 F 2 "LED_SMD:LED_0603_1608Metric_Pad1.05x0.95mm_HandSolder" H 11400 4850 50  0001 C CNN
 F 3 "~" H 11400 4850 50  0001 C CNN
+F 4 "Green LED" H 11400 4850 50  0001 C CNN "Description"
+F 5 "B1911PG--20D000514U1930" H 11400 4850 50  0001 C CNN "Digi-Key_PN"
+F 6 "B1911PG--20D000514U1930" H 11400 4850 50  0001 C CNN "MPN"
+F 7 "Harvatek Corporation" H 11400 4850 50  0001 C CNN "Manufacturer"
 	1    11400 4850
 	1    0    0    -1
@@
 F 2 "LED_SMD:LED_0603_1608Metric_Pad1.05x0.95mm_HandSolder" H 11400 5100 50  0001 C CNN
 F 3 "~" H 11400 5100 50  0001 C CNN
+F 4 "Green LED" H 11400 5100 50  0001 C CNN "Description"
+F 5 "B1911PG--20D000514U1930" H 11400 5100 50  0001 C CNN "Digi-Key_PN"
+F 6 "B1911PG--20D000514U1930" H 11400 5100 50  0001 C CNN "MPN"
+F 7 "Harvatek Corporation" H 11400 5100 50  0001 C CNN "Manufacturer"
 	1    11400 5100
 	1    0    0    -1
@@
 F 2 "LED_SMD:LED_0603_1608Metric_Pad1.05x0.95mm_HandSolder" H 11400 5350 50  0001 C CNN
 F 3 "~" H 11400 5350 50  0001 C CNN
+F 4 "Green LED" H 11400 5350 50  0001 C CNN "Description"
+F 5 "B1911PG--20D000514U1930" H 11400 5350 50  0001 C CNN "Digi-Key_PN"
+F 6 "B1911PG--20D000514U1930" H 11400 5350 50  0001 C CNN "MPN"
+F 7 "Harvatek Corporation" H 11400 5350 50  0001 C CNN "Manufacturer"
 	1    11400 5350
 	1    0    0    -1
@@
 F 2 "LED_SMD:LED_0603_1608Metric_Pad1.05x0.95mm_HandSolder" H 11400 5600 50  0001 C CNN
 F 3 "~" H 11400 5600 50  0001 C CNN
+F 4 "Green LED" H 11400 5600 50  0001 C CNN "Description"
+F 5 "B1911PG--20D000514U1930" H 11400 5600 50  0001 C CNN "Digi-Key_PN"
+F 6 "B1911PG--20D000514U1930" H 11400 5600 50  0001 C CNN "MPN"
+F 7 "Harvatek Corporation" H 11400 5600 50  0001 C CNN "Manufacturer"
 	1    11400 5600
 	1    0    0    -1
@@
 F 2 "LED_SMD:LED_0603_1608Metric_Pad1.05x0.95mm_HandSolder" H 11400 5850 50  0001 C CNN
 F 3 "~" H 11400 5850 50  0001 C CNN
+F 4 "Green LED" H 11400 5850 50  0001 C CNN "Description"
+F 5 "B1911PG--20D000514U1930" H 11400 5850 50  0001 C CNN "Digi-Key_PN"
+F 6 "B1911PG--20D000514U1930" H 11400 5850 50  0001 C CNN "MPN"
+F 7 "Harvatek Corporation" H 11400 5850 50  0001 C CNN "Manufacturer"
 	1    11400 5850
 	1    0    0    -1
@@
 F 2 "Diode_SMD:D_0603_1608Metric_Pad1.05x0.95mm_HandSolder" H 8800 1750 50  0001 C CNN
 F 3 "~" H 8800 1750 50  0001 C CNN
+F 4 "1N4448WSF-7DICT-ND" H 8800 1750 50  0001 C CNN "Digi-Key_PN"
+F 5 "1N4448WSF-7" H 8800 1750 50  0001 C CNN "MPN"
+F 6 "Diodes Incorporated" H 8800 1750 50  0001 C CNN "Manufacturer"
 	1    8800 1750
 	1    0    0    -1
@@
 F 2 "Diode_SMD:D_0603_1608Metric_Pad1.05x0.95mm_HandSolder" H 8800 2050 50  0001 C CNN
 F 3 "~" H 8800 2050 50  0001 C CNN
+F 4 "1N4448WSF-7DICT-ND" H 8800 2050 50  0001 C CNN "Digi-Key_PN"
+F 5 "1N4448WSF-7" H 8800 2050 50  0001 C CNN "MPN"
+F 6 "Diodes Incorporated" H 8800 2050 50  0001 C CNN "Manufacturer"
 	1    8800 2050
 	1    0    0    -1

Commit message: Added .1uF cap part numbers
Parts:
- C1, C10, C11, C12, C13, C14, C15, C16, C17, C2, C22, C23, C24, C4, C6, C7, C8, C9: Digi-Key_PN (none) -> 445-1314-1-ND; MPN (none) -> C1608X7R1H104K080AA; Manufacturer (none) -> TDK
Changed lines of the file:
@@
 F 2 "Capacitor_SMD:C_0603_1608Metric_Pad1.05x0.95mm_HandSolder" H 1838 4850 50  0001 C CNN
 F 3 "~" H 1800 5000 50  0001 C CNN
+F 4 "445-1314-1-ND" H 1800 5000 50  0001 C CNN "Digi-Key_PN"
+F 5 "C1608X7R1H104K080AA" H 1800 5000 50  0001 C CNN "MPN"
+F 6 "TDK" H 1800 5000 50  0001 C CNN "Manufacturer"
 	1    1800 5000
 	1    0    0    -1
@@
 F 2 "Capacitor_SMD:C_0603_1608Metric_Pad1.05x0.95mm_HandSolder" H 2238 4850 50  0001 C CNN
 F 3 "~" H 2200 5000 50  0001 C CNN
+F 4 "445-1314-1-ND" H 2200 5000 50  0001 C CNN "Digi-Key_PN"
+F 5 "C1608X7R1H104K080AA" H 2200 5000 50  0001 C CNN "MPN"
+F 6 "TDK" H 2200 5000 50  0001 C CNN "Manufacturer"
 	1    2200 5000
 	1    0    0    -1
@@
 F 2 "Capacitor_SMD:C_0603_1608Metric_Pad1.05x0.95mm_HandSolder" H 2638 4850 50  0001 C CNN
 F 3 "~" H 2600 5000 50  0001 C CNN
+F 4 "445-1314-1-ND" H 2600 5000 50  0001 C CNN "Digi-Key_PN"
+F 5 "C1608X7R1H104K080AA" H 2600 5000 50  0001 C CNN "MPN"
+F 6 "TDK" H 2600 5000 50  0001 C CNN "Manufacturer"
 	1    2600 5000
 	1    0    0    -1
@@
 F 2 "Capacitor_SMD:C_0603_1608Metric_Pad1.05x0.95mm_HandSolder" H 3038 4850 50  0001 C CNN
 F 3 "~" H 3000 5000 50  0001 C CNN
+F 4 "445-1314-1-ND" H 3000 5000 50  0001 C CNN "Digi-Key_PN"
+F 5 "C1608X7R1H104K080AA" H 3000 5000 50  0001 C CNN "MPN"
+F 6 "TDK" H 3000 5000 50  0001 C CNN "Manufacturer"
 	1    3000 5000
 	1    0    0    -1
@@
 F 2 "Capacitor_SMD:C_0603_1608Metric_Pad1.05x0.95mm_HandSolder" H 3438 4850 50  0001 C CNN
 F 3 "~" H 3400 5000 50  0001 C CNN
+F 4 "445-1314-1-ND" H 3400 5000 50  0001 C CNN "Digi-Key_PN"
+F 5 "C1608X7R1H104K080AA" H 3400 5000 50  0001 C CNN "MPN"
+F 6 "TDK" H 3400 5000 50  0001 C CNN "Manufacturer"
 	1    3400 5000
 	1    0    0    -1
@@
 F 2 "Capacitor_SMD:C_0603_1608Metric_Pad1.05x0.95mm_HandSolder" H 3838 4850 50  0001 C CNN
 F 3 "~" H 3800 5000 50  0001 C CNN
+F 4 "445-1314-1-ND" H 3800 5000 50  0001 C CNN "Digi-Key_PN"
+F 5 "C1608X7R1H104K080AA" H 3800 5000 50  0001 C CNN "MPN"
+F 6 "TDK" H 3800 5000 50  0001 C CNN "Manufacturer"
 	1    3800 5000
 	1    0    0    -1
@@
 F 2 "Capacitor_SMD:C_0603_1608Metric_Pad1.05x0.95mm_HandSolder" H 4238 4850 50  0001 C CNN
 F 3 "~" H 4200 5000 50  0001 C CNN
+F 4 "445-1314-1-ND" H 4200 5000 50  0001 C CNN "Digi-Key_PN"
+F 5 "C1608X7R1H104K080AA" H 4200 5000 50  0001 C CNN "MPN"
+F 6 "TDK" H 4200 5000 50  0001 C CNN "Manufacturer"
 	1    4200 5000
 	1    0    0    -1
@@
 F 2 "Capacitor_SMD:C_0603_1608Metric_Pad1.05x0.95mm_HandSolder" H 4638 4850 50  0001 C CNN
 F 3 "~" H 4600 5000 50  0001 C CNN
+F 4 "445-1314-1-ND" H 4600 5000 50  0001 C CNN "Digi-Key_PN"
+F 5 "C1608X7R1H104K080AA" H 4600 5000 50  0001 C CNN "MPN"
+F 6 "TDK" H 4600 5000 50  0001 C CNN "Manufacturer"
 	1    4600 5000
 	1    0    0    -1
@@
 F 2 "Capacitor_SMD:C_0603_1608Metric_Pad1.05x0.95mm_HandSolder" H 10838 1250 50  0001 C CNN
 F 3 "~" H 10800 1400 50  0001 C CNN
+F 4 "445-1314-1-ND" H 10800 1400 50  0001 C CNN "Digi-Key_PN"
+F 5 "C1608X7R1H104K080AA" H 10800 1400 50  0001 C CNN "MPN"
+F 6 "TDK" H 10800 1400 50  0001 C CNN "Manufacturer"
 	1    10800 1400
 	1    0    0    -1
@@
 F 2 "Capacitor_SMD:C_0603_1608Metric_Pad1.05x0.95mm_HandSolder" H 11688 2050 50  0001 C CNN
 F 3 "~" H 11650 2200 50  0001 C CNN
+F 4 "445-1314-1-ND" H 11650 2200 50  0001 C CNN "Digi-Key_PN"
+F 5 "C1608X7R1H104K080AA" H 11650 2200 50  0001 C CNN "MPN"
+F 6 "TDK" H 11650 2200 50  0001 C CNN "Manufacturer"
 	1    11650 2200
 	1    0    0    -1
@@
 F 2 "Capacitor_SMD:C_0603_1608Metric_Pad1.05x0.95mm_HandSolder" H 11688 1500 50  0001 C CNN
 F 3 "~" H 11650 1650 50  0001 C CNN
+F 4 "445-1314-1-ND" H 11650 1650 50  0001 C CNN "Digi-Key_PN"
+F 5 "C1608X7R1H104K080AA" H 11650 1650 50  0001 C CNN "MPN"
+F 6 "TDK" H 11650 1650 50  0001 C CNN "Manufacturer"
 	1    11650 1650
 	1    0    0    -1
@@
 F 2 "Capacitor_SMD:C_0603_1608Metric_Pad1.05x0.95mm_HandSolder" H 5438 4850 50  0001 C CNN
 F 3 "~" H 5400 5000 50  0001 C CNN
+F 4 "445-1314-1-ND" H 5400 5000 50  0001 C CNN "Digi-Key_PN"
+F 5 "C1608X7R1H104K080AA" H 5400 5000 50  0001 C CNN "MPN"
+F 6 "TDK" H 5400 5000 50  0001 C CNN "Manufacturer"
 	1    5400 5000
 	1    0    0    -1
@@
 F 2 "Capacitor_SMD:C_0603_1608Metric_Pad1.05x0.95mm_HandSolder" H 5838 4850 50  0001 C CNN
 F 3 "~" H 5800 5000 50  0001 C CNN
+F 4 "445-1314-1-ND" H 5800 5000 50  0001 C CNN "Digi-Key_PN"
+F 5 "C1608X7R1H104K080AA" H 5800 5000 50  0001 C CNN "MPN"
+F 6 "TDK" H 5800 5000 50  0001 C CNN "Manufacturer"
 	1    5800 5000
 	1    0    0    -1
@@
 F 2 "Capacitor_SMD:C_0603_1608Metric_Pad1.05x0.95mm_HandSolder" H 6238 4850 50  0001 C CNN
 F 3 "~" H 6200 5000 50  0001 C CNN
+F 4 "445-1314-1-ND" H 6200 5000 50  0001 C CNN "Digi-Key_PN"
+F 5 "C1608X7R1H104K080AA" H 6200 5000 50  0001 C CNN "MPN"
+F 6 "TDK" H 6200 5000 50  0001 C CNN "Manufacturer"
 	1    6200 5000
 	1    0    0    -1
@@
 F 2 "Capacitor_SMD:C_0603_1608Metric_Pad1.05x0.95mm_HandSolder" H 6638 4850 50  0001 C CNN
 F 3 "~" H 6600 5000 50  0001 C CNN
+F 4 "445-1314-1-ND" H 6600 5000 50  0001 C CNN "Digi-Key_PN"
+F 5 "C1608X7R1H104K080AA" H 6600 5000 50  0001 C CNN "MPN"
+F 6 "TDK" H 6600 5000 50  0001 C CNN "Manufacturer"
 	1    6600 5000
 	1    0    0    -1
@@
 F 2 "Capacitor_SMD:C_0603_1608Metric_Pad1.05x0.95mm_HandSolder" H 1438 4850 50  0001 C CNN
 F 3 "~" H 1400 5000 50  0001 C CNN
+F 4 "445-1314-1-ND" H 1400 5000 50  0001 C CNN "Digi-Key_PN"
+F 5 "C1608X7R1H104K080AA" H 1400 5000 50  0001 C CNN "MPN"
+F 6 "TDK" H 1400 5000 50  0001 C CNN "Manufacturer"
 	1    1400 5000
 	1    0    0    -1
@@
 F 2 "Capacitor_SMD:C_0603_1608Metric_Pad1.05x0.95mm_HandSolder" H 1038 4850 50  0001 C CNN
 F 3 "~" H 1000 5000 50  0001 C CNN
+F 4 "445-1314-1-ND" H 1000 5000 50  0001 C CNN "Digi-Key_PN"
+F 5 "C1608X7R1H104K080AA" H 1000 5000 50  0001 C CNN "MPN"
+F 6 "TDK" H 1000 5000 50  0001 C CNN "Manufacturer"
 	1    1000 5000
 	1    0    0    -1
@@
 F 2 "Capacitor_SMD:C_0603_1608Metric_Pad1.05x0.95mm_HandSolder" H 12138 6850 50  0001 C CNN
 F 3 "~" H 12100 7000 50  0001 C CNN
+F 4 "445-1314-1-ND" H 12100 7000 50  0001 C CNN "Digi-Key_PN"
+F 5 "C1608X7R1H104K080AA" H 12100 7000 50  0001 C CNN "MPN"
+F 6 "TDK" H 12100 7000 50  0001 C CNN "Manufacturer"
 	1    12100 7000
 	1    0    0    -1
